Commit message: add inertia to links

File: diffrobot_description/urdf/diffrobot.urdf (robot description, URDF)
Before this commit: robot diffrobot, 9 links, 8 joints
Links:
- link laser: mass None -> 0.1
- link robot_footprint: mass None -> 0.0

Commit message: fix spawn issue

File: diffrobot_description/urdf/diffrobot.urdf (robot description, URDF)
Before this commit: robot diffrobot, 9 links, 8 joints
Links:
- link robot_footprint: mass 0.0 -> None

Commit message: separate caster links and add friction

File: diffrobot_description/urdf/diffrobot.urdf (robot description, URDF)
Before this commit: robot diffrobot, 9 links, 8 joints
Links:
- link back_caster: mass 0.0 -> 0.2
- link front_caster: mass 0.0 -> 0.2

Commit message: add link for laser data

File: diffrobot_description/urdf/diffrobot.urdf (robot description, URDF)
Before this commit: robot diffrobot, 9 links, 8 joints
Links:
- added link diffrobot/laser/rp_laser, mass 0.2
Joints:
- added joint rp_laser_joint: type fixed, parent laser, child diffrobot/laser/rp_laser, origin xyz=0.0 0.0 0.0 rpy=0.0 0 0

Commit message: add gazebo xacro file for beetlebot with material and friction properties

File: diffrobot_description/urdf/diffrobot.urdf (robot description, URDF)
Before this commit: robot diffrobot, 10 links, 9 joints
Links:
- removed link back_caster
- removed link diffrobot/laser/rp_laser
- removed link imu_link
- removed link laser
- removed link left_wheel
- removed link lidar_link
- removed link right_wheel
- removed link robot_footprint
- added link beetlebot
- added link camera; collision box ; visual box 
- added link left_bar; collision cylinder ; visual cylinder 
- added link lidar; collision cylinder ; visual cylinder 
- added link rear_bar; collision cylinder ; visual cylinder 
- added link rear_caster; collision sphere ; visual sphere 
- added link right_bar; collision cylinder ; visual cylinder 
- added link top_base; collision cylinder ; visual cylinder 
- added link wheel_left; collision cylinder ; visual cylinder 
- added link wheel_right; collision cylinder ; visual cylinder 
- link base_link: mass 5.0 -> None; geometry collision cylinder ; visual cylinder 
- link front_caster: mass 0.2 -> None; geometry collision sphere ; visual sphere 
Joints:
- removed joint back_caster_joint
- removed joint front_caster_joint
- removed joint imu_joint
- removed joint laser_data_joint
- removed joint lidar_joint
- removed joint robot_footprint_joint
- removed joint rp_laser_joint
- removed joint wheel_left_joint
- removed joint wheel_right_joint
- added joint base_link_to_camera: type revolute, parent , child , axis 
- added joint base_link_to_front_caster: type ball, parent , child 
- added joint base_link_to_left_bar: type fixed, parent , child 
- added joint base_link_to_lidar: type fixed, parent , child 
- added joint base_link_to_rear_bar: type fixed, parent , child 
- added joint base_link_to_rear_caster: type ball, parent , child 
- added joint base_link_to_right_bar: type fixed, parent , child 
- added joint base_link_to_top_base: type fixed, parent , child 
- added joint base_link_to_wheel_left: type revolute, parent , child , axis 
- added joint base_link_to_wheel_right: type revolute, parent , child , axis 
- added joint footprint_to_base: type fixed, parent , child 
