Commit message: refactor: update beetlebot launch files and URDF configuration for improved robot simulation

File: beetlebot_description/urdf/beetlebot.xacro (robot description, xacro)
@@ -145,5 +145,5 @@
     </link>
     <!-- Front Caster Joint -->
-    <joint name="base_link_to_front_caster" type="continuous">
+    <joint name="base_link_to_front_caster" type="fixed">
         <parent link="base_link"/>
         <child link="front_caster"/>
@@ -175,5 +175,5 @@
     </link>
     <!-- Rear Caster Joint -->
-    <joint name="base_link_to_rear_caster" type="continuous">
+    <joint name="base_link_to_rear_caster" type="fixed">
         <parent link="base_link"/>
         <child link="rear_caster"/>

Commit message: update beetlebot URDF: add inertial properties and correct wheel joint axis

File: beetlebot_description/urdf/beetlebot.xacro (robot description, xacro)
@@ -4,4 +4,9 @@
         <link name="beetlebot">
             <pose relative_to='__model__'>0 0 0.0 0 0 0</pose>
+            <inertial>
+                <origin xyz="0 0 0.3" rpy="0 0 0"/>
+                <mass value="5"/>
+                <inertia ixx="1.5417" ixy="0" ixz="0" iyy="3.467" iyz="0" izz="4.742"/>
+            </inertial>
         </link>
         <joint name="footprint_to_base" type="fixed">
@@ -60,5 +65,5 @@
         <child link="wheel_right"/>
         <origin xyz="0 -0.33 -0.05" rpy="1.5707963267948963 0 0"/>
-        <axis xyz="0 1 0"/>
+        <axis xyz="0 0 1"/>
     </joint>
     <!-- Left Wheel Link -->
@@ -90,5 +95,5 @@
         <child link="wheel_left"/>
         <origin xyz="0 0.33 -0.05" rpy="1.5707963267948963 0 0"/>
-        <axis xyz="0 1 0"/>
+        <axis xyz="0 0 1"/>
     </joint>
     <!-- Top Base Link -->

Commit message: fix beetlebot wheel joint axis orientation in URDF

File: beetlebot_description/urdf/beetlebot.xacro (robot description, xacro)
@@ -65,5 +65,5 @@
         <child link="wheel_right"/>
         <origin xyz="0 -0.33 -0.05" rpy="1.5707963267948963 0 0"/>
-        <axis xyz="0 0 1"/>
+        <axis xyz="0 0 -1"/>
     </joint>
     <!-- Left Wheel Link -->
@@ -95,5 +95,5 @@
         <child link="wheel_left"/>
         <origin xyz="0 0.33 -0.05" rpy="1.5707963267948963 0 0"/>
-        <axis xyz="0 0 1"/>
+        <axis xyz="0 0 -1"/>
     </joint>
     <!-- Top Base Link -->

Commit message: add IMU link and joint to Beetlebot URDF; update ROS bridge for IMU topic

File: beetlebot_description/urdf/beetlebot.xacro (robot description, xacro)
@@ -333,3 +333,32 @@
         <limit lower="-1.14" upper="1.14" velocity="3.14" effort="10.0"/>
     </joint>
+    <!-- IMU Link -->
+    <link name="imu_link">
+        <visual>
+            <origin xyz="0 0 0" rpy="0 0 0"/>
+            <geometry>
+                <box size="0.05 0.05 0.05"/>
+            </geometry>
+            <material name="camera_material">
+                <color rgba="0.015996293361446288 0.22696587349938613 0.07036009568874305 1"/>
+            </material>
+        </visual>
+        <collision>
+            <origin xyz="0 0 0" rpy="0 0 0"/>
+            <geometry>
+                <box size="0.05 0.05 0.05"/>
+            </geometry>
+        </collision>
+        <inertial>
+            <origin xyz="0 0 0" rpy="0 0 0"/>
+            <mass value="1"/>
+            <inertia ixx="0.16666666666666666" ixy="0" ixz="0" iyy="0.16666666666666666" iyz="0" izz="0.16666666666666666"/>
+        </inertial>
+    </link>
+    <!-- Camera Joint -->
+    <joint name="imu_joint" type="fixed">
+        <parent link="base_link"/>
+        <child link="imu_link"/>
+        <origin xyz="0.3 0 0.34" rpy="0 0 0"/>
+    </joint>
     </robot>

Commit message: add IMU link and joint to beetlebot.xacro for enhanced sensor integration

File: beetlebot_description/urdf/beetlebot.xacro (robot description, xacro)
@@ -334,3 +334,32 @@
         <limit lower="-1.14" upper="1.14" velocity="3.14" effort="10.0"/>
     </joint>
+    <!-- IMU Link -->
+    <link name="imu_link">
+        <visual>
+            <origin xyz="0 0 0" rpy="0 0 0"/>
+            <geometry>
+                <box size="0.05 0.05 0.05"/>
+            </geometry>
+            <material name="camera_material">
+                <color rgba="0.015996293361446288 0.22696587349938613 0.07036009568874305 1"/>
+            </material>
+        </visual>
+        <collision>
+            <origin xyz="0 0 0" rpy="0 0 0"/>
+            <geometry>
+                <box size="0.05 0.05 0.05"/>
+            </geometry>
+        </collision>
+        <inertial>
+            <origin xyz="0 0 0" rpy="0 0 0"/>
+            <mass value="1"/>
+            <inertia ixx="0.16666666666666666" ixy="0" ixz="0" iyy="0.16666666666666666" iyz="0" izz="0.16666666666666666"/>
+        </inertial>
+    </link>
+    <!-- IMU Joint -->
+    <joint name="imu_joint" type="fixed">
+        <parent link="base_link"/>
+        <child link="imu_link"/>
+        <origin xyz="0.3 0 0.34" rpy="0 0 0"/>
+    </joint>
     </robot>
